File: doc/resources/conn.kicad_pcb (KiCad board)
At the start: 2 copper layers, 26 x 18 mm, 6 parts, among them J1 IN, J2 OUT, J3 POGO, J4 Molex

Commit message: Implement tab creation from user-provided lines
Other:
- board text added: "TabPosition"
Changed lines of the file:
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@@
-(kicad_pcb (version 20171130) (host pcbnew 5.1.5-52549c5~86~ubuntu19.10.1)
+(kicad_pcb (version 20171130) (host pcbnew 5.1.5+dfsg1-2build2)
   (general
     (thickness 1.6)
-    (drawings 13)
+    (drawings 21)
     (tracks 156)
     (zones 0)
@@
       (net 7 7))
   )
+  (gr_text TabPosition (at 141 71) (layer Eco1.User)
+    (effects (font (size 1 1) (thickness 0.15)))
+  )
+  (gr_text TabPosition (at 96 64) (layer Eco1.User)
+    (effects (font (size 1 1) (thickness 0.15)))
+  )
+  (gr_line (start 103 64) (end 107 64) (layer Eco1.User) (width 0.15))
+  (gr_line (start 134 71) (end 130 71) (layer Eco1.User) (width 0.15))
+  (gr_text TabPosition (at 125 82) (layer Eco2.User)
+    (effects (font (size 1 1) (thickness 0.15)))
+  )
+  (gr_text TabPosition (at 112 53) (layer Eco2.User)
+    (effects (font (size 1 1) (thickness 0.15)))
+  )
+  (gr_line (start 125 79) (end 125 76) (layer Eco2.User) (width 0.15))
+  (gr_line (start 112 57) (end 112 60) (layer Eco2.User) (width 0.15))
   (gr_text "PogoPads\nv0.2 9/2019\nro.fi.muni.cz" (at 118.5 70.5) (layer B.SilkS)
     (effects (font (size 1.5 1.5) (thickness 0.3)) (justify mirror))

Commit message: Start CLI reimplementation
Parts:
- added REF**: Tab, kikit:Tab, F.Cu at (110.5, 59.0)
- added REF**: Tab, kikit:Tab, F.Cu at (105.5, 73.0)
- added REF**: Tab, kikit:Tab, F.Cu at (118.5, 77.0)
- added REF**: Tab, kikit:Tab, F.Cu at (131.5, 63.0)
Other:
- board text removed: "TabPosition"

Commit message: Draft implementation of tabs via annotations
Parts:
- removed the REF** at (110.5, 59.0)
- removed the REF** at (131.5, 63.0)
- added REF**: Tab, kikit:Tab, F.Cu at (131.2, 76.5)
- added REF**: Tab, kikit:Tab, F.Cu at (110.5, 58.8)
- added REF**: Tab, kikit:Tab, F.Cu at (131.8, 63.0)
- moved REF** 0.25 mm to (105.2, 73.0)
- moved REF** 0.25 mm to (118.5, 77.2)

Commit message: Prepare new examples, fix corresponding bugs
Parts:
- removed the REF** at (131.2, 76.5)
Changed lines of the file:
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@@
     (tracks 156)
     (zones 0)
-    (modules 11)
+    (modules 10)
     (nets 11)
   )
@@
   )
   (module kikit:Tab (layer F.Cu)
-    (at 131.25 76.5 135)
-    (descr "A symbol representing annotation for tab placement")
-    (attr virtual)
-    (fp_text reference REF** (at 0 -2 135) (layer F.SilkS) hide
-      (effects (font (size 1 1) (thickness 0.15)))
-    )
-    (fp_text value Tab (at -3 -1 135) (layer Dwgs.User)
-      (effects (font (size 1.2 1.2) (thickness 0.2)))
-    )
-    (fp_line (start 0.25 1) (end 0.25 -1) (layer Dwgs.User) (width 0.3))
-    (fp_line (start 0.25 0) (end -2.75 0) (layer Dwgs.User) (width 0.3))
-    (fp_line (start 0.25 0) (end -0.75 -1) (layer Dwgs.User) (width 0.3))
-    (fp_line (start 0.25 0) (end -0.75 1) (layer Dwgs.User) (width 0.3))
-    (fp_text user "KIKIT: width: 3mm" (at -5.5 0 45) (layer Dwgs.User)
-      (effects (font (size 1 1) (thickness 0.15)))
-    )
-  )
-  (module kikit:Tab (layer F.Cu)
