File: test/resources/multiboard.kicad_pcb (KiCad board)
At the start: 2 copper layers, 120 x 20 mm, 3 parts

Commit message: Add option to preserve annotation
Parts:
- added REF**: Tab, kikit:Tab, F.Cu at (147.0, 89.5)
Changed lines of the file:
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@@
-(kicad_pcb (version 20171130) (host pcbnew 5.1.9-73d0e3b20d~88~ubuntu20.04.1)
+(kicad_pcb (version 20171130) (host pcbnew 5.1.12-84ad8e8a86~92~ubuntu20.04.1)
   (general
     (thickness 1.6)
@@
     (tracks 0)
     (zones 0)
-    (modules 3)
+    (modules 4)
     (nets 1)
   )
@@
     (uvia_drill 0.1)
   )
+  (module kikit:Tab (layer F.Cu)
+    (at 147 89.5 270)
+    (descr "A symbol representing annotation for tab placement")
+    (attr virtual)
+    (fp_text reference REF** (at 0 -2 90) (layer F.SilkS) hide
+      (effects (font (size 1 1) (thickness 0.15)))
+    )
+    (fp_text value Tab (at -2.75 -1 90) (layer Dwgs.User)
+      (effects (font (size 1.2 1.2) (thickness 0.2)))
+    )
+    (fp_text user "KIKIT: width: 3mm" (at -5.5 0) (layer Dwgs.User)
+      (effects (font (size 1 1) (thickness 0.15)))
+    )
+    (fp_line (start 0.25 0) (end -0.75 1) (layer Dwgs.User) (width 0.3))
+    (fp_line (start 0.25 0) (end -0.75 -1) (layer Dwgs.User) (width 0.3))
+    (fp_line (start 0.25 0) (end -2.75 0) (layer Dwgs.User) (width 0.3))
+    (fp_line (start 0.25 1) (end 0.25 -1) (layer Dwgs.User) (width 0.3))
+  )
   (module kikit:Board (layer F.Cu)
     (at 185 90)
     (descr "Mark board for extraction")
     (fp_text reference B3 (at -4.5 -5) (layer Dwgs.User)
+      (effects (font (size 1 1) (thickness 0.15)) (justify left))
+    )
+    (fp_text value Board (at -7.25 -5) (layer Dwgs.User)
+      (effects (font (size 1 1) (thickness 0.15)))
+    )
+    (fp_line (start 0 0) (end -1 -0.5) (layer Dwgs.User) (width 0.2))
+    (fp_line (start 0 0) (end 0.5 -1) (layer Dwgs.User) (width 0.2))
+    (fp_line (start -1.25 -4) (end -9.25 -4) (layer Dwgs.User) (width 0.2))
+    (fp_line (start 0 0) (end -1.25 -4) (layer Dwgs.User) (width 0.2))
+  )
+  (module kikit:Board (layer F.Cu)
+    (at 135 90)
+    (descr "Mark board for extraction")
+    (fp_text reference B2 (at -4.5 -5) (layer Dwgs.User)
       (effects (font (size 1 1) (thickness 0.15)) (justify left))
     )
@@
   )
   (module kikit:Board (layer F.Cu)
-    (at 135 90)
+    (at 100 90)
     (descr "Mark board for extraction")
-    (fp_text reference B2 (at -4.5 -5) (layer Dwgs.User)
+    (fp_text reference B1 (at -4.5 -5) (layer Dwgs.User)
       (effects (font (size 1 1) (thickness 0.15)) (justify left))
     )
@@
     (fp_line (start 0 0) (end -1.25 -4) (layer Dwgs.User) (width 0.2))
   )
-  (module kikit:Board (layer F.Cu)
-    (at 100 90)
-    (descr "Mark board for extraction")
-    (fp_text reference B1 (at -4.5 -5) (layer Dwgs.User)
-      (effects (font (size 1 1) (thickness 0.15)) (justify left))
-    )
-    (fp_text value Board (at -7.25 -5) (layer Dwgs.User)
-      (effects (font (size 1 1) (thickness 0.15)))
-    )
-    (fp_line (start 0 0) (end -1.25 -4) (layer Dwgs.User) (width 0.2))
-    (fp_line (start -1.25 -4) (end -9.25 -4) (layer Dwgs.User) (width 0.2))
-    (fp_line (start 0 0) (end 0.5 -1) (layer Dwgs.User) (width 0.2))
-    (fp_line (start 0 0) (end -1 -0.5) (layer Dwgs.User) (width 0.2))
-  )
   (gr_text C (at 185 100) (layer F.SilkS)
